File: stm32f103_core.sch (KiCad schematic (older format))
At the start: 39 parts, among them SW1 SW_Push, SW2 SW_Push

Commit message: update,
Parts:
- removed C? (x6): C, symbol Device:C
- removed J? (x2): Conn_01x02, symbol Connector_Generic:Conn_01x02
- removed R? (x2): R, symbol Device:R
- added J1: JMP_USER_BTN_EN, Button_Switch_THT:SW_PUSH_6mm_H4.3mm, symbol Connector_Generic:Conn_02x01
- added J3: Conn_02x01, footprint-lib.pretty:Pin_Header_Straight_1x02_Pitch2.54mm, symbol Connector_Generic:Conn_02x01
- C1, C2: renamed from C?; value C -> 104; footprint (none) -> Capacitor_SMD:C_0603_1608Metric_Pad1.05x0.95mm_HandSolder
- C3: renamed from C?; footprint (none) -> Capacitor_SMD:C_0603_1608Metric_Pad1.05x0.95mm_HandSolder
- C4, C5: renamed from C?; value C -> 200; footprint (none) -> Capacitor_SMD:C_0603_1608Metric_Pad1.05x0.95mm_HandSolder
- C6, C7: renamed from C?; value C -> 150; footprint (none) -> Capacitor_SMD:C_0603_1608Metric_Pad1.05x0.95mm_HandSolder
- J2: renamed from J?; footprint (none) -> Connector_PinHeader_2.54mm:PinHeader_1x05_P2.54mm_Vertical
- Q1: renamed from Q?; value Q_PNP_BCE -> PNP8550
- R1, R3, R6, R7: renamed from R?; footprint (none) -> Resistor_SMD:R_0603_1608Metric_Pad1.05x0.95mm_HandSolder
- R10: renamed from R?; value R -> 152; footprint (none) -> Resistor_SMD:R_0603_1608Metric_Pad1.05x0.95mm_HandSolder
- R11, R12, R14, R9: renamed from R?; value R -> 0; footprint (none) -> Resistor_SMD:R_0603_1608Metric_Pad1.05x0.95mm_HandSolder
- R13: renamed from R?; value R -> 103; footprint (none) -> Resistor_SMD:R_0603_1608Metric_Pad1.05x0.95mm_HandSolder
- R2: renamed from R?; value R -> 472; footprint (none) -> Resistor_SMD:R_0603_1608Metric_Pad1.05x0.95mm_HandSolder
- R4, R5: renamed from R?; value R -> 100; footprint (none) -> Resistor_SMD:R_0603_1608Metric_Pad1.05x0.95mm_HandSolder
- R8: renamed from R?; value R -> 22R; footprint (none) -> Resistor_SMD:R_0603_1608Metric_Pad1.05x0.95mm_HandSolder
- SW1: value SW_Push -> RESET_BTN; footprint (none) -> Button_Switch_SMD:SW_SPST_FSMSM
- SW2: value SW_Push -> USER_BTN; footprint (none) -> Button_Switch_SMD:SW_SPST_FSMSM
- U1: renamed from U?; footprint (none) -> Package_DFN_QFN:QFN-48-1EP_7x7mm_P0.5mm_EP5.15x5.15mm
- Y1: renamed from Y?; footprint (none) -> w_crystal:hc-49_smd
- Y2: renamed from Y?; footprint (none) -> w_crystal:crystal_smd_ma-505
- gave numbers to parts that had none: 1
Connections:
- net labels added: AGND, PA0, PA10, PA13, PA14, PA15, PA4, PA5, PA6, PA7, PA8, PA9, PB0, PB10, PB12, PB13, PB14, PB15, PB2, PB3, PB4, PB5, PB6, PB7, PB8, PB9, PC0, PC1, PC10, PC10_TX, PC11, PC11_RX, PC12, PC14, PC15, PC2, PC3, PC4, PC5, PC6, PC7, PC8, PC9
- wire segments 127 -> 145
Other:
- moved on the sheet: SW1, SW2
