File: virtual_com_port_interface.sch (KiCad schematic (older format))
At the start: 5 parts

Commit message: update,
Parts:
- D1, D2: renamed from D?; footprint (none) -> LED_SMD:LED_0805_2012Metric_Pad1.15x1.40mm_HandSolder
- R15, R16: renamed from R?; footprint (none) -> Resistor_SMD:R_0603_1608Metric_Pad1.05x0.95mm_HandSolder
- gave numbers to parts that had none: 1
Changed lines of the file:
@@
 EESchema Schematic File Version 4
+LIBS:stm32f103_core-cache
 EELAYER 26 0
 EELAYER END
 $Descr A4 11693 8268
 encoding utf-8
-Sheet 2 2
+Sheet 2 5
 Title ""
 Date ""
@@
 $EndDescr
 $Comp
-L customized_power:+3V3 #PWR?
+L customized_power:+3V3 #PWR0112
 U 1 1 5BC809B5
 P 1200 2350
-F 0 "#PWR?" H 1200 2200 50  0001 C CNN
+F 0 "#PWR0112" H 1200 2200 50  0001 C CNN
 F 1 "+3V3" H 1250 2550 50  0000 C CNN
 F 2 "" H 1200 2350 50  0001 C CNN
@@
 $EndComp
 $Comp
-L Device:R R?
+L Device:R R15
 U 1 1 5BC809EC
 P 1200 2800
-F 0 "R?" H 1300 2850 50  0000 L CNN
+F 0 "R15" H 1300 2850 50  0000 L CNN
 F 1 "R" H 1300 2800 50  0000 L CNN
-F 2 "" V 1130 2800 50  0001 C CNN
+F 2 "Resistor_SMD:R_0603_1608Metric_Pad1.05x0.95mm_HandSolder" V 1130 2800 50  0001 C CNN
 F 3 "~" H 1200 2800 50  0001 C CNN
 	1    1200 2800
@@
 $EndComp
 $Comp
-L Device:R R?
+L Device:R R16
 U 1 1 5BC80A3C
 P 1500 2800
-F 0 "R?" H 1600 2850 50  0000 L CNN
+F 0 "R16" H 1600 2850 50  0000 L CNN
 F 1 "R" H 1600 2800 50  0000 L CNN
-F 2 "" V 1430 2800 50  0001 C CNN
+F 2 "Resistor_SMD:R_0603_1608Metric_Pad1.05x0.95mm_HandSolder" V 1430 2800 50  0001 C CNN
 F 3 "~" H 1500 2800 50  0001 C CNN
 	1    1500 2800
@@
 $EndComp
 $Comp
-L Device:LED D?
+L Device:LED D1
 U 1 1 5BC80AA9
 P 1200 3200
-F 0 "D?" V 1250 3050 50  0000 R CNN
+F 0 "D1" V 1250 3050 50  0000 R CNN
 F 1 "LED" V 1150 3050 50  0000 R CNN
-F 2 "" H 1200 3200 50  0001 C CNN
+F 2 "LED_SMD:LED_0805_2012Metric_Pad1.15x1.40mm_HandSolder" H 1200 3200 50  0001 C CNN
 F 3 "~" H 1200 3200 50  0001 C CNN
 	1    1200 3200
@@
 $EndComp
 $Comp
-L Device:LED D?
+L Device:LED D2
 U 1 1 5BC80AE1
 P 1500 3200
-F 0 "D?" V 1550 3050 50  0000 R CNN
+F 0 "D2" V 1550 3050 50  0000 R CNN
 F 1 "LED" V 1450 3050 50  0000 R CNN
-F 2 "" H 1500 3200 50  0001 C CNN
+F 2 "LED_SMD:LED_0805_2012Metric_Pad1.15x1.40mm_HandSolder" H 1500 3200 50  0001 C CNN
 F 3 "~" H 1500 3200 50  0001 C CNN
 	1    1500 3200
@@
 	1500 3750 1500 3350
 $Comp
-L taobao-components:CP2102GMR U?
+L taobao-components:CP2102GMR U2
 U 1 1 5BC819A8
 P 6350 3050
-F 0 "U?" H 6350 4050 50  0000 C CNN
+F 0 "U2" H 6350 4050 50  0000 C CNN
 F 1 "CP2102GMR" H 6350 3950 50  0000 C CNN
 F 2 "" H 6350 3050 50  0001 C CNN
