File: stm32f103-core.kicad_pcb (KiCad board)
At the start: 2 copper layers, 32 parts, among them J1 Conn_01x12, J3 Conn_01x12, J4 Conn_01x12, SW1 SW_Push, U1 STM32F103C8T6, U2 AMS1117-3.3, U3 USB_PCB, Y1 O8M, Y2 O32.768K

Commit message: update,
Parts:
- removed U3: USB_PCB, footprint-lib:usb-PCB
- J4: footprint Connector_PinHeader_1.27mm:PinHeader_1x12_P1.27mm_Vertical -> Connector_PinHeader_1.27mm:PinHeader_1x20_P1.27mm_Vertical
- moved J4 10.3 mm to (30.2, 31.9)
- moved D1 3.50 mm to (23.1, 31.4)
- moved D2 3.50 mm to (27.4, 31.5)
- moved JP1 3.50 mm to (22.4, 26.1)
- moved JP2 3.50 mm to (25.2, 26.1)
- moved R1 3.50 mm to (20.3, 24.7)
- moved R2 3.50 mm to (27.6, 25.1)
- moved R3 3.50 mm to (21.0, 31.2)
- moved R5 3.50 mm to (25.5, 31.3)
- moved C1 0.50 mm to (19.2, 21.4), turned to 180 degrees
Connections:
- J4 pad 1: /PA0 -> Net-(J4-Pad1)
- J4 pad 10: /PB1 -> /PA1
- J4 pad 11: /PB10 -> /PA2
- J4 pad 12: /PB11 -> /PA3
- J4 pad 2: /PA1 -> GND
- J4 pad 3: /PA2 -> Net-(J4-Pad3)
- J4 pad 4: /PA3 -> Net-(J4-Pad4)
- J4 pad 5: /PA4 -> Net-(J4-Pad5)
- J4 pad 6: /PA5 -> Net-(J4-Pad6)
- J4 pad 7: /PA6 -> Net-(J4-Pad7)
- J4 pad 8: /PA7 -> Net-(J4-Pad8)
- J4 pad 9: /PB0 -> /PA0
- JP3 pad 1: Net-(JP3-Pad1) -> Net-(J4-Pad1)
Routing:
- net Net-(JP3-Pad1): track 27.9 -> 0.00 mm
- net Net-(J4-Pad1): track 0.00 -> 23.6 mm
- net 3V3: track 133.0 -> 124.3 mm
- net GND: track 153.6 -> 146.5 mm, vias 7 -> 6
- net /BOOT0: track 23.9 -> 27.8 mm
- net Net-(D2-Pad1): track 4.11 -> 1.96 mm
- net /BOOT1: track 24.4 -> 22.5 mm
- net /PA7: track 16.3 -> 14.5 mm
- net /PB1: track 11.1 -> 10.4 mm

Commit message: update,
Parts:
- moved R2 21.0 mm to (26.8, 4.10), turned to 180 degrees
- moved JP2 19.8 mm to (25.5, 6.30), turned to 0 degrees
- moved U2 18.0 mm to (24.1, 33.6)
- moved JP3 17.8 mm to (30.2, 35.5), turned to 270 degrees
- moved C6 8.94 mm to (21.5, 28.9)
- moved R5 7.25 mm to (22.6, 24.6)
- moved D1 6.80 mm to (25.1, 24.9)
- moved R1 6.75 mm to (24.4, 19.4), turned to 180 degrees
- moved D2 6.59 mm to (27.2, 24.9)
- moved R3 6.55 mm to (20.8, 24.7)
- moved C7 5.22 mm to (17.8, 32.5), turned to 90 degrees
- moved JP1 5.08 mm to (24.8, 21.6), turned to 0 degrees
- moved C9 2.82 mm to (17.8, 28.9)
- moved SW1 1.84 mm to (14.9, 26.9)
- moved C3 1.78 mm to (9.98, 17.4)
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Routing:
- net Net-(J4-Pad1): track 23.6 -> 2.88 mm
- net +5V: track 24.3 -> 32.1 mm
- net /BOOT0: track 27.8 -> 20.5 mm
- net /BOOT1: track 22.5 -> 15.4 mm
- net Net-(D1-Pad1): track 2.12 -> 6.15 mm
- net Net-(D2-Pad1): track 1.96 -> 5.45 mm
- net 3V3: track 124.3 -> 121.2 mm, vias 7 -> 5
- net /RESET: track 19.2 -> 16.3 mm
- net /OSCOUT: track 24.3 -> 25.7 mm
- net GND: track 146.5 -> 145.7 mm, vias 6 -> 7
- net /PB8: track 11.6 -> 12.2 mm
- net /PB12: track 7.58 -> 8.22 mm
- net /PB13: track 7.06 -> 7.66 mm
- net /PB9: track 12.1 -> 12.6 mm

Commit message: update,
Parts:
- moved C5 23.7 mm to (24.7, 44.6), turned to 180 degrees
- moved C12 17.2 mm to (16.3, 37.1), turned to 270 degrees
- moved C13 16.2 mm to (13.0, 37.1), turned to 270 degrees
- moved C11 14.6 mm to (14.7, 39.7)
- moved C10 14.5 mm to (14.7, 41.3)
- moved C9 14.1 mm to (27.8, 39.0)
- moved J4 14.1 mm to (40.2, 41.9)
- moved Y1 14.1 mm to (20.1, 37.7)
- moved C1 14.1 mm to (29.2, 31.4)
- moved C3 14.1 mm to (20.0, 27.4)
- moved C4 14.1 mm to (22.6, 18.1)
- moved C8 14.1 mm to (20.0, 29.2)
- moved J3 14.1 mm to (33.8, 13.4)
- moved JP2 14.1 mm to (35.5, 16.3)
- moved R4 14.1 mm to (27.8, 35.5)
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Connections:
- J4 pad 3: Net-(J4-Pad3) -> 3V3
Routing:
- net +5V: track 32.1 -> 15.3 mm
- net 3V3: track 121.2 -> 109.4 mm
- net GND: track 145.7 -> 154.7 mm, vias 7 -> 15
- net /PC15: track 21.5 -> 15.2 mm
- net Net-(J4-Pad1): track 2.88 -> 5.20 mm
- net /PC14: track 19.7 -> 17.8 mm
- net /OSCIN: track 20.5 -> 18.9 mm
- net /PA1: track 13.2 -> 14.7 mm
- net /PA0: track 14.7 -> 15.8 mm
- net Net-(D2-Pad1): track 5.45 -> 6.30 mm
- net Net-(D1-Pad1): track 6.15 -> 6.80 mm
- net /BOOT0: track 20.5 -> 19.8 mm
- added copper zone on B.Cu, net GND
- added copper zone on F.Cu, net GND
Other:
- board outline added: 30 x 35 mm
