File: stm32f103-core.kicad_pcb (KiCad board)
At the start: 2 copper layers, 30 x 35 mm, 31 parts, among them J1 Conn_01x14, J3 Conn_01x12, J4 Conn_01x12, SW1 SW_Push, U1 STM32F103C8T6, U2 AMS1117-3.3, Y1 O8M, Y2 O32.768K

Commit message: update,
Parts:
- moved Y1 1.50 mm to (20.1, 38.2)
Routing:
- net 3V3: track 114.4 -> 130.7 mm
- net GND: track 137.2 -> 144.3 mm, vias 25 -> 26
- net /SWIO: track 15.6 -> 16.9 mm
- net /PC15: track 23.1 -> 23.7 mm
- net /PC14: track 24.9 -> 25.5 mm
Other:
- net class 3v3 added: clearance 0.2, trace_width 0.75, via_dia 1, via_drill 0.4
- net class Default: via_dia 0.8 -> 0.5
- net class GND: trace_width 1 -> 0.75; via_dia 1.2 -> 1

Commit message: update,
Parts:
- C5, C6: footprint Capacitor_Tantalum_SMD:CP_EIA-2012-12_Kemet-R_Pad1.30x1.05mm_HandSolder -> Capacitor_Tantalum_SMD:CP_EIA-3216-12_Kemet-S_Pad1.58x1.35mm_HandSolder
- Y1: footprint Crystal:Crystal_SMD_HC49-SD -> w_crystal:hc-49_smd
- Y2: footprint Crystal:Crystal_SMD_MicroCrystal_CC7V-T1A-2Pin_3.2x1.5mm_HandSoldering -> footprint-lib.pretty:MC-306
- moved Y2 9.90 mm to (5.00, 37.1)
Connections:
- net 3V3 renamed +3V3
- J1 pad 13: (no net) -> Net-(J1-Pad13)
- J3 pad 10: (no net) -> Net-(J3-Pad10)
- J3 pad 11: (no net) -> Net-(J3-Pad11)
- J3 pad 12: (no net) -> Net-(J3-Pad12)
- J4 pad 4: (no net) -> Net-(J4-Pad4)
- J4 pad 5: (no net) -> Net-(J4-Pad5)
- J4 pad 6: (no net) -> Net-(J4-Pad6)
- J4 pad 7: (no net) -> Net-(J4-Pad7)
- J4 pad 8: (no net) -> Net-(J4-Pad8)
- U1 pad 1: (no net) -> /VBAT
Routing:
- net 3V3: track 0.00 -> 130.7 mm, vias 0 -> 5
- net +3V3: track 130.7 -> 0.00 mm, vias 5 -> 0

Commit message: update,
Parts:
- moved Y2 4.56 mm to (5.41, 32.6), turned to 0 degrees
Connections:
- Y2 pad 2: /PC14 -> (no net)
- Y2 pad 4: (no net) -> /PC14
Changed lines of the file:
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@@
     (add_net +5V)
+  )
+  (module footprint-lib.pretty:MC-306 (layer F.Cu)
+    (at 5.4102 32.5628)
+    (descr "<b>MC-306 CRYSTAL UNIT</b><p>Source: MC-306_405_406_E07X.PDF")
+    (attr smd)
+    (fp_text reference Y2 (at -1.48071 -3.45353) (layer F.SilkS)
+      (effects (font (size 1.00102 1.00102) (thickness 0.05)))
+    )
+    (fp_text value O32.768K (at -0.84523 3.9628) (layer F.SilkS)
+      (effects (font (size 1.00121 1.00121) (thickness 0.05)))
+    )
+    (fp_line (start -3.9 -1.5) (end 3.9 -1.5) (layer Dwgs.User) (width 0.2032))
+    (fp_line (start 3.9 1.5) (end -3.9 1.5) (layer Dwgs.User) (width 0.2032))
+    (fp_line (start -1.4 -1.5) (end 1.4 -1.5) (layer F.SilkS) (width 0.2032))
+    (fp_line (start 1.4 1.5) (end -1.4 1.5) (layer F.SilkS) (width 0.2032))
+    (fp_arc (start -3.8 0) (end -3.8 0.5) (angle -180) (layer F.SilkS) (width 0.2032))
+    (pad 1 smd rect (at -2.75 1.6) (size 1.3 1.9) (layers F.Cu F.Paste F.Mask)
+      (net 10 /PC15))
+    (pad 2 smd rect (at 2.75 1.6) (size 1.3 1.9) (layers F.Cu F.Paste F.Mask))
+    (pad 3 smd rect (at 2.75 -1.6 180) (size 1.3 1.9) (layers F.Cu F.Paste F.Mask))
+    (pad 4 smd rect (at -2.75 -1.6 180) (size 1.3 1.9) (layers F.Cu F.Paste F.Mask)
+      (net 9 /PC14))
+    (model /home/logic/_workspace/kicad/kicad_library/kicad-packages3d/Crystal_SMD_SeikoEpson_MC306-4pin_8.0x3.2mm.wrl
+      (at (xyz 0 0 0))
+      (scale (xyz 1 1 1))
+      (rotate (xyz 0 0 0))
+    )
+    (model /home/logic/_workspace/kicad/kicad_library/kicad-packages3d/Crystal_SMD_SeikoEpson_MC306-4pin_8.0x3.2mm_HandSoldering.wrl
+      (at (xyz 0 0 0))
+      (scale (xyz 1 1 1))
+      (rotate (xyz 0 0 0))
+    )
   )
   (module Capacitor_Tantalum_SMD:CP_EIA-3216-12_Kemet-S_Pad1.58x1.35mm_HandSolder (layer F.Cu)
@@
       (net 3 GND))
     (model ${KISYS3DMOD}/Capacitor_Tantalum_SMD.3dshapes/CP_EIA-3216-12_Kemet-S.wrl
-      (at (xyz 0 0 0))
-      (scale (xyz 1 1 1))
-      (rotate (xyz 0 0 0))
-    )
-  )
-  (module footprint-lib.pretty:MC-306 (layer F.Cu)
-    (at 5 37.1 180)
-    (descr "<b>MC-306 CRYSTAL UNIT</b><p>Source: MC-306_405_406_E07X.PDF")
-    (attr smd)
-    (fp_text reference Y2 (at -1.48071 -3.45353 180) (layer F.SilkS)
-      (effects (font (size 1.00102 1.00102) (thickness 0.05)))
-    )
-    (fp_text value O32.768K (at -0.84523 3.9628 180) (layer F.SilkS)
-      (effects (font (size 1.00121 1.00121) (thickness 0.05)))
-    )
-    (fp_line (start -3.9 -1.5) (end 3.9 -1.5) (layer Dwgs.User) (width 0.2032))
-    (fp_line (start 3.9 1.5) (end -3.9 1.5) (layer Dwgs.User) (width 0.2032))
-    (fp_line (start -1.4 -1.5) (end 1.4 -1.5) (layer F.SilkS) (width 0.2032))
-    (fp_line (start 1.4 1.5) (end -1.4 1.5) (layer F.SilkS) (width 0.2032))
-    (fp_arc (start -3.8 0) (end -3.8 0.5) (angle -180) (layer F.SilkS) (width 0.2032))
-    (pad 1 smd rect (at -2.75 1.6 180) (size 1.3 1.9) (layers F.Cu F.Paste F.Mask)
-      (net 10 /PC15))
-    (pad 2 smd rect (at 2.75 1.6 180) (size 1.3 1.9) (layers F.Cu F.Paste F.Mask)
-      (net 9 /PC14))
-    (pad 3 smd rect (at 2.75 -1.6) (size 1.3 1.9) (layers F.Cu F.Paste F.Mask))
-    (pad 4 smd rect (at -2.75 -1.6) (size 1.3 1.9) (layers F.Cu F.Paste F.Mask))
-    (model /home/logic/_workspace/kicad/kicad_library/kicad-packages3d/Crystal_SMD_SeikoEpson_MC306-4pin_8.0x3.2mm.wrl
-      (at (xyz 0 0 0))
-      (scale (xyz 1 1 1))
-      (rotate (xyz 0 0 0))
-    )
-    (model /home/logic/_workspace/kicad/kicad_library/kicad-packages3d/Crystal_SMD_SeikoEpson_MC306-4pin_8.0x3.2mm_HandSoldering.wrl
       (at (xyz 0 0 0))
       (scale (xyz 1 1 1))
@@
   (gr_line (start 0 100) (end 100 100) (layer Dwgs.User) (width 0.2))
   (gr_line (start 0 0) (end 0 100) (layer Dwgs.User) (width 0.2))
-  (segment (start 40.2 38.12) (end 40.52 38.12) (width 0.25) (layer F.Cu) (net 54) (status 30))
   (segment (start 31.45 19.05) (end 31.6 18.9) (width 0.5) (layer F.Cu) (net 1) (status 30))
   (segment (start 31.45 20.65) (end 31.45 19.05) (width 0.25) (layer F.Cu) (net 1) (status 30))
@@
   (segment (start 14.3 36.3) (end 14.075 36.3) (width 0.25) (layer F.Cu) (net 9))
   (segment (start 14.3 36.3) (end 14.2 36.4) (width 0.25) (layer F.Cu) (net 9))
+  (segment (start 24.64004 30.15996) (end 25.35 29.45) (width 0.25) (layer F.Cu) (net 9))
+  (segment (start 18.09004 30.15996) (end 24.64004 30.15996) (width 0.25) (layer F.Cu) (net 9))
   (segment (start 25.35 29.45) (end 25.35 27.75) (width 0.25) (layer F.Cu) (net 9))
-  (segment (start 24.6 30.2) (end 25.35 29.45) (width 0.25) (layer F.Cu) (net 9))
-  (segment (start 18.05 30.2) (end 24.6 30.2) (width 0.25) (layer F.Cu) (net 9))
-  (segment (start 16.7 31.55) (end 18.05 30.2) (width 0.25) (layer F.Cu) (net 9))
+  (segment (start 16.7 34.6) (end 16.7 31.55) (width 0.25) (layer F.Cu) (net 9))
   (segment (start 14.8 36.3) (end 14.9 36.2) (width 0.25) (layer F.Cu) (net 9))
-  (segment (start 14.3 36.3) (end 14.8 36.3) (width 0.25) (layer F.Cu) (net 9))
-  (segment (start 14.9 35.7) (end 15.1 35.5) (width 0.25) (layer F.Cu) (net 9))
-  (segment (start 15.8 35.5) (end 16.7 34.6) (width 0.25) (layer F.Cu) (net 9))
-  (segment (start 16.7 34.6) (end 16.7 31.55) (width 0.25) (layer F.Cu) (net 9))
   (segment (start 14.9 36.2) (end 14.9 35.7) (width 0.25) (layer F.Cu) (net 9))
   (segment (start 15.1 35.5) (end 15.8 35.5) (width 0.25) (layer F.Cu) (net 9))
+  (segment (start 16.7 31.55) (end 18.09004 30.15996) (width 0.25) (layer F.Cu) (net 9))
+  (segment (start 14.9 35.7) (end 15.1 35.5) (width 0.25) (layer F.Cu) (net 9))
+  (segment (start 14.3 36.3) (end 14.8 36.3) (width 0.25) (layer F.Cu) (net 9))
+  (segment (start 15.8 35.5) (end 16.7 34.6) (width 0.25) (layer F.Cu) (net 9))
   (segment (start 16.6 37.175) (end 16.525 37.1) (width 0.25) (layer F.Cu) (net 10))
   (segment (start 17.2 36.425) (end 16.525 37.1) (width 0.25) (layer F.Cu) (net 10))
@@
   (segment (start 35.925 15.875) (end 35.5 16.3) (width 0.25) (layer F.Cu) (net 47) (status 30))
   (segment (start 35.925 14.1) (end 35.925 15.875) (width 0.25) (layer F.Cu) (net 47) (status 30))
+  (segment (start 40.2 38.12) (end 40.52 38.12) (width 0.25) (layer F.Cu) (net 54) (status 30))
   (zone (net 3) (net_name GND) (layer F.Cu) (hatch edge 0.508)
     (connect_pads (clearance 0.426))

Commit message: update,
Parts:
- added D3: LED_GREEN, LED_SMD:LED_0805_2012Metric_Pad1.15x1.40mm_HandSolder, F.Cu at (6.10, 22.5)
- added R6: R511, Resistor_SMD:R_0603_1608Metric_Pad1.05x0.95mm_HandSolder, F.Cu at (5.85, 24.3)
Connections:
- U1 pad 1: /VBAT -> +3V3
Changed lines of the file:
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@@
     (tracks 513)
     (zones 0)
-    (modules 31)
+    (modules 33)
     (nets 59)
   )
@@
   (net 47 "Net-(BOOT1-Pad2)")
   (net 48 +3V3)
-  (net 49 /VBAT)
-  (net 50 "Net-(J4-Pad8)")
-  (net 51 "Net-(J4-Pad7)")
-  (net 52 "Net-(J4-Pad6)")
-  (net 53 "Net-(J4-Pad5)")
-  (net 54 "Net-(J4-Pad4)")
-  (net 55 "Net-(J1-Pad13)")
-  (net 56 "Net-(J3-Pad12)")
-  (net 57 "Net-(J3-Pad11)")
-  (net 58 "Net-(J3-Pad10)")
+  (net 49 "Net-(J4-Pad8)")
+  (net 50 "Net-(J4-Pad7)")
+  (net 51 "Net-(J4-Pad6)")
+  (net 52 "Net-(J4-Pad5)")
+  (net 53 "Net-(J4-Pad4)")
+  (net 54 "Net-(J1-Pad13)")
+  (net 55 "Net-(J3-Pad12)")
+  (net 56 "Net-(J3-Pad11)")
+  (net 57 "Net-(J3-Pad10)")
+  (net 58 "Net-(D3-Pad1)")
   (net_class Default "This is the default net class."
     (clearance 0.2)
@@
     (add_net /SWCLK)
     (add_net /SWIO)
-    (add_net /VBAT)
     (add_net "Net-(BOOT0-Pad2)")
     (add_net "Net-(BOOT1-Pad2)")
     (add_net "Net-(D1-Pad1)")
     (add_net "Net-(D2-Pad1)")
+    (add_net "Net-(D3-Pad1)")
     (add_net "Net-(J1-Pad13)")
     (add_net "Net-(J3-Pad10)")
@@
     (uvia_drill 0.1)
     (add_net +5V)
+  )
+  (module LED_SMD:LED_0805_2012Metric_Pad1.15x1.40mm_HandSolder (layer F.Cu)
+    (at 6.095761 22.549041)
+    (descr "LED SMD 0805 (2012 Metric), square (rectangular) end terminal, IPC_7351 nominal, (Body size source: https://docs.google.com/spreadsheets/d/1BsfQQcO9C6DZCsRaXUlFlo91Tg2WpOkGARC1WS5S8t0/edit?usp=sharing), generated with kicad-footprint-generator")
+    (tags "LED handsolder")
+    (attr smd)
+    (fp_text reference D3 (at 0 -1.65) (layer F.SilkS)
+      (effects (font (size 1 1) (thickness 0.15)))
+    )
+    (fp_text value LED_GREEN (at 0 1.65) (layer F.Fab)
+      (effects (font (size 1 1) (thickness 0.15)))
+    )
+    (fp_line (start 1 -0.6) (end -0.7 -0.6) (layer F.Fab) (width 0.1))
+    (fp_line (start -0.7 -0.6) (end -1 -0.3) (layer F.Fab) (width 0.1))
+    (fp_line (start -1 -0.3) (end -1 0.6) (layer F.Fab) (width 0.1))
+    (fp_line (start -1 0.6) (end 1 0.6) (layer F.Fab) (width 0.1))
+    (fp_line (start 1 0.6) (end 1 -0.6) (layer F.Fab) (width 0.1))
+    (fp_line (start 1 -0.96) (end -1.86 -0.96) (layer F.SilkS) (width 0.12))
+    (fp_line (start -1.86 -0.96) (end -1.86 0.96) (layer F.SilkS) (width 0.12))
+    (fp_line (start -1.86 0.96) (end 1 0.96) (layer F.SilkS) (width 0.12))
+    (fp_line (start -1.85 0.95) (end -1.85 -0.95) (layer F.CrtYd) (width 0.05))
+    (fp_line (start -1.85 -0.95) (end 1.85 -0.95) (layer F.CrtYd) (width 0.05))
+    (fp_line (start 1.85 -0.95) (end 1.85 0.95) (layer F.CrtYd) (width 0.05))
+    (fp_line (start 1.85 0.95) (end -1.85 0.95) (layer F.CrtYd) (width 0.05))
+    (fp_text user %R (at 0 0) (layer F.Fab)
+      (effects (font (size 0.5 0.5) (thickness 0.08)))
+    )
+    (pad 1 smd roundrect (at -1.025 0) (size 1.15 1.4) (layers F.Cu F.Paste F.Mask) (roundrect_rratio 0.217391)
+      (net 58 "Net-(D3-Pad1)"))
+    (pad 2 smd roundrect (at 1.025 0) (size 1.15 1.4) (layers F.Cu F.Paste F.Mask) (roundrect_rratio 0.217391)
+      (net 8 /PC13))
+    (model ${KISYS3DMOD}/LED_SMD.3dshapes/LED_0805_2012Metric.wrl
+      (at (xyz 0 0 0))
+      (scale (xyz 1 1 1))
+      (rotate (xyz 0 0 0))
+    )
+  )
+  (module Resistor_SMD:R_0603_1608Metric_Pad1.05x0.95mm_HandSolder (layer F.Cu)
+    (at 5.850761 24.324041)
+    (descr "Resistor SMD 0603 (1608 Metric), square (rectangular) end terminal, IPC_7351 nominal with elongated pad for handsoldering. (Body size source: http://www.tortai-tech.com/upload/download/2011102023233369053.pdf), generated with kicad-footprint-generator")
+    (tags "resistor handsolder")
+    (attr smd)
+    (fp_text reference R6 (at 0 -1.43) (layer F.SilkS)
+      (effects (font (size 1 1) (thickness 0.15)))
+    )
+    (fp_text value R511 (at 0 1.43) (layer F.Fab)
+      (effects (font (size 1 1) (thickness 0.15)))
+    )
+    (fp_line (start -0.8 0.4) (end -0.8 -0.4) (layer F.Fab) (width 0.1))
+    (fp_line (start -0.8 -0.4) (end 0.8 -0.4) (layer F.Fab) (width 0.1))
+    (fp_line (start 0.8 -0.4) (end 0.8 0.4) (layer F.Fab) (width 0.1))
+    (fp_line (start 0.8 0.4) (end -0.8 0.4) (layer F.Fab) (width 0.1))
+    (fp_line (start -0.171267 -0.51) (end 0.171267 -0.51) (layer F.SilkS) (width 0.12))
+    (fp_line (start -0.171267 0.51) (end 0.171267 0.51) (layer F.SilkS) (width 0.12))
+    (fp_line (start -1.65 0.73) (end -1.65 -0.73) (layer F.CrtYd) (width 0.05))
+    (fp_line (start -1.65 -0.73) (end 1.65 -0.73) (layer F.CrtYd) (width 0.05))
+    (fp_line (start 1.65 -0.73) (end 1.65 0.73) (layer F.CrtYd) (width 0.05))
+    (fp_line (start 1.65 0.73) (end -1.65 0.73) (layer F.CrtYd) (width 0.05))
+    (fp_text user %R (at 0 0) (layer F.Fab)
+      (effects (font (size 0.4 0.4) (thickness 0.06)))
+    )
+    (pad 1 smd roundrect (at -0.875 0) (size 1.05 0.95) (layers F.Cu F.Paste F.Mask) (roundrect_rratio 0.25)
+      (net 58 "Net-(D3-Pad1)"))
+    (pad 2 smd roundrect (at 0.875 0) (size 1.05 0.95) (layers F.Cu F.Paste F.Mask) (roundrect_rratio 0.25)
+      (net 3 GND))
+    (model ${KISYS3DMOD}/Resistor_SMD.3dshapes/R_0603_1608Metric.wrl
+      (at (xyz 0 0 0))
+      (scale (xyz 1 1 1))
+      (rotate (xyz 0 0 0))
+    )
   )
   (module footprint-lib.pretty:MC-306 (layer F.Cu)
@@
       (net 13 /PA0))
     (pad 8 thru_hole oval (at 0 8.89 180) (size 1 1) (drill 0.65) (layers *.Cu *.Mask)
-      (net 50 "Net-(J4-Pad8)"))
+      (net 49 "Net-(J4-Pad8)"))
     (pad 7 thru_hole oval (at 0 7.62 180) (size 1 1) (drill 0.65) (layers *.Cu *.Mask)
-      (net 51 "Net-(J4-Pad7)"))
+      (net 50 "Net-(J4-Pad7)"))
     (pad 6 thru_hole oval (at 0 6.35 180) (size 1 1) (drill 0.65) (layers *.Cu *.Mask)
-      (net 52 "Net-(J4-Pad6)"))
+      (net 51 "Net-(J4-Pad6)"))
     (pad 5 thru_hole oval (at 0 5.08 180) (size 1 1) (drill 0.65) (layers *.Cu *.Mask)
-      (net 53 "Net-(J4-Pad5)"))
+      (net 52 "Net-(J4-Pad5)"))
     (pad 4 thru_hole oval (at 0 3.81 180) (size 1 1) (drill 0.65) (layers *.Cu *.Mask)
-      (net 54 "Net-(J4-Pad4)"))
+      (net 53 "Net-(J4-Pad4)"))
     (pad 3 thru_hole oval (at 0 2.54 180) (size 1 1) (drill 0.65) (layers *.Cu *.Mask)
       (net 48 +3V3))
@@
       (net 34 /PB9))
     (pad 13 thru_hole oval (at 0 15.24) (size 1 1) (drill 0.65) (layers *.Cu *.Mask)
-      (net 55 "Net-(J1-Pad13)"))
+      (net 54 "Net-(J1-Pad13)"))
     (pad 14 thru_hole oval (at 0 16.51) (size 1 1) (drill 0.65) (layers *.Cu *.Mask)
       (net 8 /PC13))
@@
     (fp_line (start -0.525 -0.635) (end 1.05 -0.635) (layer F.Fab) (width 0.1))
     (pad 12 thru_hole oval (at 0 13.97 270) (size 1 1) (drill 0.65) (layers *.Cu *.Mask)
-      (net 56 "Net-(J3-Pad12)"))
+      (net 55 "Net-(J3-Pad12)"))
     (pad 11 thru_hole oval (at 0 12.7 270) (size 1 1) (drill 0.65) (layers *.Cu *.Mask)
-      (net 57 "Net-(J3-Pad11)"))
+      (net 56 "Net-(J3-Pad11)"))
     (pad 10 thru_hole oval (at 0 11.43 270) (size 1 1) (drill 0.65) (layers *.Cu *.Mask)
-      (net 58 "Net-(J3-Pad10)"))
+      (net 57 "Net-(J3-Pad10)"))
     (pad 9 thru_hole oval (at 0 10.16 270) (size 1 1) (drill 0.65) (layers *.Cu *.Mask)
       (net 44 /PA12))
@@
       (net 8 /PC13))
     (pad 1 smd rect (at -4.35 -2.75 90) (size 1.3 0.25) (layers F.Cu F.Paste F.Mask)
-      (net 49 /VBAT))
+      (net 48 +3V3))
     (model ${KISYS3DMOD}/Package_QFP.3dshapes/LQFP-48_7x7mm_P0.5mm.wrl
       (at (xyz 0 0 0))
@@
   (segment (start 35.925 15.875) (end 35.5 16.3) (width 0.25) (layer F.Cu) (net 47) (status 30))
   (segment (start 35.925 14.1) (end 35.925 15.875) (width 0.25) (layer F.Cu) (net 47) (status 30))
-  (segment (start 40.2 38.12) (end 40.52 38.12) (width 0.25) (layer F.Cu) (net 54) (status 30))
+  (segment (start 40.2 38.12) (end 40.52 38.12) (width 0.25) (layer F.Cu) (net 53) (status 30))
   (zone (net 3) (net_name GND) (layer F.Cu) (hatch edge 0.508)
     (connect_pads (clearance 0.426))

Commit message: update,
Parts:
- moved R6 14.5 mm to (16.1, 14.1), turned to 270 degrees
- moved D3 14.4 mm to (17.9, 14.3), turned to 270 degrees
- moved Y2 9.61 mm to (14.8, 34.6), turned to 90 degrees
- moved J4 4.00 mm to (40.2, 37.9)
- moved J1 4.00 mm to (13.6, 13.7)
- moved C3 1.65 mm to (19.3, 28.1), turned to 0 degrees
- moved C8 1.20 mm to (19.3, 26.5), turned to 0 degrees
- moved BOOT1 1.00 mm to (34.5, 16.3)
Routing:
- net +3V3: track 0.00 -> 172.6 mm, vias 0 -> 7
- net 3V3: track 130.7 -> 0.00 mm, vias 5 -> 0
- net GND: track 144.3 -> 167.0 mm, vias 26 -> 23
- net /PC13: track 15.4 -> 35.2 mm, vias 0 -> 1
- net /PA15: track 9.85 -> 18.6 mm
- net /PB11: track 10.3 -> 14.2 mm
- net Net-(J4-Pad1): track 2.74 -> 6.64 mm
- net /PB5: track 12.8 -> 9.24 mm
- net /PB10: track 10.0 -> 13.6 mm
- net /PB1: track 9.91 -> 13.0 mm
- net /SWCLK: track 9.39 -> 12.5 mm
- net /PB8: track 13.2 -> 10.2 mm
- net /PB9: track 13.7 -> 10.8 mm
- net /PB6: track 12.4 -> 9.47 mm
- net /PB0: track 9.74 -> 12.6 mm
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
Commit message: update,
Other:
- net class 3v3 removed
- net class Default removed
- net class GND removed
- net class PWR removed
