File: stm32f103-core.sch (KiCad schematic (older format))
At the start: 32 parts, among them J1 Conn_01x12, J3 Conn_01x12, J4 Conn_01x12, SW1 SW_Push, U1 STM32F103C8T6, U2 AMS1117-3.3, U3 USB_PCB, Y1 O8M, Y2 O32.768K

Commit message: update,
Parts:
- removed U3: USB_PCB, footprint-lib:usb-PCB, symbol taobao-components:USB_PCB
- J4: footprint Connector_PinHeader_1.27mm:PinHeader_1x12_P1.27mm_Vertical -> Connector_PinHeader_1.27mm:PinHeader_1x20_P1.27mm_Vertical; symbol Connector_Generic:Conn_01x12 -> Connector_Generic:Conn_01x20
Other:
- moved on the sheet: JP3
Changed lines of the file:
@@
 Connection ~ 12900 5000
-$Comp
-L taobao-components:USB_PCB U3
-U 1 1 5BD566CF
-P 12050 6750
-F 0 "U3" H 12019 7165 50  0000 C CNN
-F 1 "USB_PCB" H 12019 7074 50  0000 C CNN
-F 2 "footprint-lib:usb-PCB" H 12050 6800 50  0001 C CNN
-F 3 "" H 12050 6800 50  0001 C CNN
-	1    12050 6750
-	-1   0    0    -1
-$EndComp
 $Comp
 L tinkerforge:+5V #PWR0126
 U 1 1 5BD5A319
-P 12950 6450
-F 0 "#PWR0126" H 12950 6300 50  0001 C CNN
-F 1 "+5V" H 12965 6623 50  0000 C CNN
-F 2 "" H 12950 6450 50  0000 C CNN
-F 3 "" H 12950 6450 50  0000 C CNN
-	1    12950 6450
-	1    0    0    -1
+P 4200 4950
+F 0 "#PWR0126" H 4200 4800 50  0001 C CNN
+F 1 "+5V" H 4215 5123 50  0000 C CNN
+F 2 "" H 4200 4950 50  0000 C CNN
+F 3 "" H 4200 4950 50  0000 C CNN
+	1    4200 4950
+	-1   0    0    1
 $EndComp
 $Comp
 L power:GND #PWR0127
 U 1 1 5BD5A437
-P 12550 7450
-F 0 "#PWR0127" H 12550 7200 50  0001 C CNN
-F 1 "GND" H 12555 7277 50  0000 C CNN
-F 2 "" H 12550 7450 50  0001 C CNN
-F 3 "" H 12550 7450 50  0001 C CNN
-	1    12550 7450
-	1    0    0    -1
-$EndComp
-Wire Wire Line
-	12400 6900 12550 6900
-Wire Wire Line
-	12950 6600 12950 6450
+P 3850 4750
+F 0 "#PWR0127" H 3850 4500 50  0001 C CNN
+F 1 "GND" H 3855 4577 50  0000 C CNN
+F 2 "" H 3850 4750 50  0001 C CNN
+F 3 "" H 3850 4750 50  0001 C CNN
+	1    3850 4750
+	1    0    0    -1
+$EndComp
+Wire Wire Line
+	4200 4800 4200 4950
 $Comp
 L tinkerforge:3V3 #PWR0128
@@
 $EndComp
 $Comp
-L Connector_Generic:Conn_01x12 J4
+L Connector_Generic:Conn_01x20 J4
 U 1 1 5BDCE49F
-P 4950 3500
+P 4950 3900
 F 0 "J4" H 4869 2675 50  0000 C CNN
 F 1 "Conn_01x12" H 4869 2766 50  0000 C CNN
-F 2 "Connector_PinHeader_1.27mm:PinHeader_1x12_P1.27mm_Vertical" H 4950 3500 50  0001 C CNN
-F 3 "~" H 4950 3500 50  0001 C CNN
-	1    4950 3500
+F 2 "Connector_PinHeader_1.27mm:PinHeader_1x20_P1.27mm_Vertical" H 4950 3900 50  0001 C CNN
+F 3 "~" H 4950 3900 50  0001 C CNN
+	1    4950 3900
 	1    0    0    1
 $EndComp
-Wire Wire Line
-	12550 6900 12550 7450
 Text Label 10400 4550 1    50   ~ 0
 VCC3V3
@@
 L Device:Jumper_NO_Small JP3
 U 1 1 5BE05EFF
-P 12700 6600
-F 0 "JP3" H 12700 6785 50  0000 C CNN
-F 1 "Jumper_NO_Small" H 12700 6694 50  0000 C CNN
-F 2 "Jumper:SolderJumper-2_P1.3mm_Open_TrianglePad1.0x1.5mm" H 12700 6600 50  0001 C CNN
-F 3 "~" H 12700 6600 50  0001 C CNN
-	1    12700 6600
-	1    0    0    -1
-$EndComp
-Wire Wire Line
-	12400 6600 12600 6600
-Wire Wire Line
-	12800 6600 12950 6600
+P 4450 4800
+F 0 "JP3" H 4450 4985 50  0000 C CNN
+F 1 "Jumper_NO_Small" H 4450 4894 50  0000 C CNN
+F 2 "Jumper:SolderJumper-2_P1.3mm_Open_TrianglePad1.0x1.5mm" H 4450 4800 50  0001 C CNN
+F 3 "~" H 4450 4800 50  0001 C CNN
+	1    4450 4800
+	-1   0    0    1
+$EndComp
+Wire Wire Line
+	4750 4800 4550 4800
+Wire Wire Line
+	4350 4800 4200 4800
 Text Label 2000 3600 2    50   ~ 0
 PB9
@@
 Wire Wire Line
 	4350 3800 4750 3800
+Wire Wire Line
+	3850 4750 3850 4700
+Wire Wire Line
+	3850 4700 4750 4700
 $EndSCHEMATC

Commit message: update,
Connections:
- net 3V3: now also J4.3 (Pin_3)
Changed lines of the file:
@@
 Wire Wire Line
 	3850 4700 4750 4700
+$Comp
+L tinkerforge:3V3 #PWR?
+U 1 1 5BF0CF31
+P 3950 4550
+F 0 "#PWR?" H 3950 4400 50  0001 C CNN
+F 1 "3V3" H 3965 4723 50  0000 C CNN
+F 2 "" H 3950 4550 50  0000 C CNN
+F 3 "" H 3950 4550 50  0000 C CNN
+	1    3950 4550
+	1    0    0    -1
+$EndComp
+Wire Wire Line
+	3950 4550 3950 4600
+Wire Wire Line
+	3950 4600 4750 4600
 $EndSCHEMATC
