File: stm32f103-core.sch (KiCad schematic (older format))
At the start: 31 parts, among them J1 Conn_01x14, J3 Conn_01x12, J4 Conn_01x12, SW1 SW_Push, U1 STM32F103C8T6, U2 AMS1117-3.3, Y1 O8M, Y2 O32.768K

Commit message: update,
Parts:
- renumbered JP1 to BOOT0, JP2 to BOOT1
Changed lines of the file:
@@
 	14500 3100 14500 3350
 $Comp
-L Jumper:SolderJumper_3_Open JP1
+L Jumper:SolderJumper_3_Open BOOT0
 U 1 1 5BCF8FA5
 P 11800 2850
-F 0 "JP1" V 11754 2918 50  0000 L CNN
+F 0 "BOOT0" V 11754 2918 50  0000 L CNN
 F 1 "SolderJumper_3_Open" V 11845 2918 50  0000 L CNN
 F 2 "Jumper:SolderJumper-3_P2.0mm_Open_TrianglePad1.0x1.5mm" H 11800 2850 50  0001 C CNN
@@
 $EndComp
 $Comp
-L Jumper:SolderJumper_3_Open JP2
+L Jumper:SolderJumper_3_Open BOOT1
 U 1 1 5BCF9021
 P 12650 2850
-F 0 "JP2" V 12604 2918 50  0000 L CNN
+F 0 "BOOT1" V 12604 2918 50  0000 L CNN
 F 1 "SolderJumper_3_Open" V 12695 2918 50  0000 L CNN
 F 2 "Jumper:SolderJumper-3_P2.0mm_Open_TrianglePad1.0x1.5mm" H 12650 2850 50  0001 C CNN

Commit message: update,
Parts:
- removed C5, C6: TC106,10V, Capacitor_Tantalum_SMD:CP_EIA-2012-12_Kemet-R_Pad1.30x1.05mm_HandSolder, symbol stm32f103-core-rescue:TC106,10V-taobao-tc
- added C? (x2): TC106,10V, symbol taobao-tc:TC106,10V
Connections:
- net +5V: now also C?.1
- net GND: now also C?.2, C?.2
- net 3V3 renamed +3V3
- net +3V3: now also C?.1
Other:
- moved on the sheet: C8

Commit message: update,
Parts:
- Y1: footprint Crystal:Crystal_SMD_HC49-SD -> w_crystal:hc-49_smd
Changed lines of the file:
@@
 F 0 "Y1" V 14654 6788 50  0000 L CNN
 F 1 "O8M" V 14745 6788 50  0000 L CNN
-F 2 "Crystal:Crystal_SMD_HC49-SD" H 14700 6700 50  0001 C CNN
+F 2 "w_crystal:hc-49_smd" H 14700 6700 50  0001 C CNN
 F 3 "~" H 14700 6700 50  0001 C CNN
 	1    14700 6700

Commit message: update,
Parts:
- C5, C6: renamed from C?; footprint (none) -> Capacitor_Tantalum_SMD:CP_EIA-3216-12_Kemet-S_Pad1.58x1.35mm_HandSolder
- Y2: footprint Crystal:Crystal_SMD_MicroCrystal_CC7V-T1A-2Pin_3.2x1.5mm_HandSoldering -> footprint-lib.pretty:MC-306
Changed lines of the file:
@@
 F 0 "Y2" V 14654 7588 50  0000 L CNN
 F 1 "O32.768K" V 14745 7588 50  0000 L CNN
-F 2 "Crystal:Crystal_SMD_MicroCrystal_CC7V-T1A-2Pin_3.2x1.5mm_HandSoldering" H 14700 7500 50  0001 C CNN
+F 2 "footprint-lib.pretty:MC-306" H 14700 7500 50  0001 C CNN
 F 3 "~" H 14700 7500 50  0001 C CNN
 	1    14700 7500
@@
 	2150 3700 2150 3650
 $Comp
-L power:+3V3 #PWR?
+L power:+3V3 #PWR0101
 U 1 1 5BCAC201
 P 2150 2400
-F 0 "#PWR?" H 2150 2250 50  0001 C CNN
+F 0 "#PWR0101" H 2150 2250 50  0001 C CNN
 F 1 "+3V3" H 2200 2600 50  0000 C CNN
 F 2 "" H 2150 2400 50  0001 C CNN
@@
 $EndComp
 $Comp
-L power:+3V3 #PWR?
+L power:+3V3 #PWR0103
 U 1 1 5BCACA2F
 P 3950 4550
-F 0 "#PWR?" H 3950 4400 50  0001 C CNN
+F 0 "#PWR0103" H 3950 4400 50  0001 C CNN
 F 1 "+3V3" H 4000 4750 50  0000 C CNN
 F 2 "" H 3950 4550 50  0001 C CNN
@@
 $EndComp
 $Comp
-L power:+5V #PWR?
+L power:+5V #PWR0105
 U 1 1 5BCACB86
 P 4200 4950
-F 0 "#PWR?" H 4200 4800 50  0001 C CNN
+F 0 "#PWR0105" H 4200 4800 50  0001 C CNN
 F 1 "+5V" H 4200 5150 50  0000 C CNN
 F 2 "" H 4200 4950 50  0001 C CNN
@@
 $EndComp
 $Comp
-L power:+3V3 #PWR?
+L power:+3V3 #PWR0107
 U 1 1 5BCAD5BF
 P 6300 1950
-F 0 "#PWR?" H 6300 1800 50  0001 C CNN
+F 0 "#PWR0107" H 6300 1800 50  0001 C CNN
 F 1 "+3V3" H 6350 2150 50  0000 C CNN
 F 2 "" H 6300 1950 50  0001 C CNN
@@
 $EndComp
 $Comp
-L power:+3V3 #PWR?
+L power:+3V3 #PWR0113
 U 1 1 5BCBE3DE
 P 7850 5650
-F 0 "#PWR?" H 7850 5500 50  0001 C CNN
+F 0 "#PWR0113" H 7850 5500 50  0001 C CNN
 F 1 "+3V3" H 7900 5850 50  0000 C CNN
 F 2 "" H 7850 5650 50  0001 C CNN
@@
 $EndComp
 $Comp
-L power:+3V3 #PWR?
+L power:+3V3 #PWR0114
 U 1 1 5BCE7C1D
 P 8300 5650
-F 0 "#PWR?" H 8300 5500 50  0001 C CNN
+F 0 "#PWR0114" H 8300 5500 50  0001 C CNN
 F 1 "+3V3" H 8350 5850 50  0000 C CNN
 F 2 "" H 8300 5650 50  0001 C CNN
@@
 $EndComp
 $Comp
-L power:+3V3 #PWR?
+L power:+3V3 #PWR0115
 U 1 1 5BCE7C66
 P 8700 5650
-F 0 "#PWR?" H 8700 5500 50  0001 C CNN
+F 0 "#PWR0115" H 8700 5500 50  0001 C CNN
 F 1 "+3V3" H 8750 5850 50  0000 C CNN
 F 2 "" H 8700 5650 50  0001 C CNN
@@
 $EndComp
 $Comp
-L power:+3V3 #PWR?
+L power:+3V3 #PWR0117
 U 1 1 5BCE7CAF
 P 9150 5650
-F 0 "#PWR?" H 9150 5500 50  0001 C CNN
+F 0 "#PWR0117" H 9150 5500 50  0001 C CNN
 F 1 "+3V3" H 9200 5850 50  0000 C CNN
 F 2 "" H 9150 5650 50  0001 C CNN
@@
 $EndComp
 $Comp
-L power:+3V3 #PWR?
+L power:+3V3 #PWR0119
 U 1 1 5BCE8262
 P 13000 4800
-F 0 "#PWR?" H 13000 4650 50  0001 C CNN
+F 0 "#PWR0119" H 13000 4650 50  0001 C CNN
 F 1 "+3V3" H 13050 5000 50  0000 C CNN
 F 2 "" H 13000 4800 50  0001 C CNN
@@
 $EndComp
 $Comp
-L power:+3V3 #PWR?
+L power:+3V3 #PWR0121
 U 1 1 5BCE8771
 P 14200 4750
-F 0 "#PWR?" H 14200 4600 50  0001 C CNN
+F 0 "#PWR0121" H 14200 4600 50  0001 C CNN
 F 1 "+3V3" H 14250 4950 50  0000 C CNN
 F 2 "" H 14200 4750 50  0001 C CNN
@@
 $EndComp
 $Comp
-L power:+3V3 #PWR?
+L power:+3V3 #PWR0125
 U 1 1 5BCE87BA
 P 14850 4750
-F 0 "#PWR?" H 14850 4600 50  0001 C CNN
+F 0 "#PWR0125" H 14850 4600 50  0001 C CNN
 F 1 "+3V3" H 14900 4950 50  0000 C CNN
 F 2 "" H 14850 4750 50  0001 C CNN
@@
 $EndComp
 $Comp
-L customized_power:+5V #PWR?
+L customized_power:+5V #PWR0126
 U 1 1 5BCE8D55
 P 11400 4800
-F 0 "#PWR?" H 11400 4650 50  0001 C CNN
+F 0 "#PWR0126" H 11400 4650 50  0001 C CNN
 F 1 "+5V" H 11450 5000 50  0000 C CNN
 F 2 "" H 11400 4800 50  0001 C CNN
@@
 $EndComp
 $Comp
-L taobao-tc:TC106,10V C?
+L taobao-tc:TC106,10V C5
 U 1 1 5BCE9101
 P 11550 5250
-F 0 "C?" H 11650 5300 50  0000 L CNN
+F 0 "C5" H 11650 5300 50  0000 L CNN
 F 1 "TC106,10V" H 11650 5250 50  0000 L CNN
-F 2 "" H 11550 5250 50  0001 C CNN
+F 2 "Capacitor_Tantalum_SMD:CP_EIA-3216-12_Kemet-S_Pad1.58x1.35mm_HandSolder" H 11550 5250 50  0001 C CNN
 F 3 "" H 11550 5250 50  0001 C CNN
 	1    11550 5250
@@
 $EndComp
 $Comp
-L taobao-tc:TC106,10V C?
+L taobao-tc:TC106,10V C6
 U 1 1 5BCE94BD
 P 12500 5250
-F 0 "C?" H 12600 5300 50  0000 L CNN
+F 0 "C6" H 12600 5300 50  0000 L CNN
 F 1 "TC106,10V" H 12600 5250 50  0000 L CNN
-F 2 "" H 12500 5250 50  0001 C CNN
+F 2 "Capacitor_Tantalum_SMD:CP_EIA-3216-12_Kemet-S_Pad1.58x1.35mm_HandSolder" H 12500 5250 50  0001 C CNN
 F 3 "" H 12500 5250 50  0001 C CNN
 	1    12500 5250
@@
 $EndComp
 $Comp
-L power:+3V3 #PWR?
+L power:+3V3 #PWR0128
 U 1 1 5BCF284B
 P 5950 1950
-F 0 "#PWR?" H 5950 1800 50  0001 C CNN
+F 0 "#PWR0128" H 5950 1800 50  0001 C CNN
 F 1 "+3V3" H 6000 2150 50  0000 C CNN
 F 2 "" H 5950 1950 50  0001 C CNN
@@
 $EndComp
 $Comp
-L power:+3V3 #PWR?
+L power:+3V3 #PWR0130
 U 1 1 5BCF3126
 P 14500 2200
-F 0 "#PWR?" H 14500 2050 50  0001 C CNN
+F 0 "#PWR0130" H 14500 2050 50  0001 C CNN
 F 1 "+3V3" H 14550 2400 50  0000 C CNN
 F 2 "" H 14500 2200 50  0001 C CNN
@@
 $EndComp
 $Comp
-L power:+3V3 #PWR?
+L power:+3V3 #PWR0132
 U 1 1 5BCF394E
 P 12650 2350
-F 0 "#PWR?" H 12650 2200 50  0001 C CNN
+F 0 "#PWR0132" H 12650 2200 50  0001 C CNN
 F 1 "+3V3" H 12700 2550 50  0000 C CNN
 F 2 "" H 12650 2350 50  0001 C CNN
@@
 $EndComp
 $Comp
-L power:+3V3 #PWR?
+L power:+3V3 #PWR0133
 U 1 1 5BCF3997
 P 11800 2350
-F 0 "#PWR?" H 11800 2200 50  0001 C CNN
+F 0 "#PWR0133" H 11800 2200 50  0001 C CNN
 F 1 "+3V3" H 11850 2550 50  0000 C CNN
 F 2 "" H 11800 2350 50  0001 C CNN

Commit message: update,
Parts:
- added D?: LED_GREEN, LED_SMD:LED_0805_2012Metric_Pad1.15x1.40mm_HandSolder, symbol taobao-components:LED_GREEN
- added R?: R511, Resistor_SMD:R_0603_1608Metric_Pad1.05x0.95mm_HandSolder, symbol taobao-r:R511
- Y2: symbol taobao-osc:O32.768K -> taobao-osc:O_EPSON_32.768K
Connections:
- net labels added: VDD_1, VDD_2, VSS_1, VSS_2
- wire segments 170 -> 184
Other:
- moved on the sheet: C5, C6, C7, C8, U2

Commit message: update,
Parts:
- gave numbers to parts that had none: 2
Changed lines of the file:
@@
 	5900 2250 5900 2350
 $Comp
-L power:GND #PWR?
+L power:GND #PWR0134
 U 1 1 5BDA790B
 P 5900 2950
-F 0 "#PWR?" H 5900 2700 50  0001 C CNN
+F 0 "#PWR0134" H 5900 2700 50  0001 C CNN
 F 1 "GND" H 5950 2750 50  0000 C CNN
 F 2 "" H 5900 2950 50  0001 C CNN
@@
 Connection ~ 5900 2850
 $Comp
-L taobao-components:LED_GREEN D?
+L taobao-components:LED_GREEN D3
 U 1 1 5BDD943F
 P 13550 5000
-F 0 "D?" V 13596 4932 50  0000 R CNN
+F 0 "D3" V 13596 4932 50  0000 R CNN
 F 1 "LED_GREEN" V 13505 4932 50  0000 R CNN
 F 2 "LED_SMD:LED_0805_2012Metric_Pad1.15x1.40mm_HandSolder" V 13550 5000 50  0001 C CNN
@@
 $EndComp
 $Comp
-L taobao-r:R511 R?
+L taobao-r:R511 R6
 U 1 1 5BDD9445
 P 13550 5300
-F 0 "R?" H 13609 5346 50  0000 L CNN
+F 0 "R6" H 13609 5346 50  0000 L CNN
 F 1 "R511" H 13609 5255 50  0000 L CNN
 F 2 "Resistor_SMD:R_0603_1608Metric_Pad1.05x0.95mm_HandSolder" H 13550 5300 50  0001 C CNN
@@
 $EndComp
 $Comp
-L power:GND #PWR?
+L power:GND #PWR0135
 U 1 1 5BDD944B
 P 13550 5500
-F 0 "#PWR?" H 13550 5250 50  0001 C CNN
+F 0 "#PWR0135" H 13550 5250 50  0001 C CNN
 F 1 "GND" H 13555 5327 50  0000 C CNN
 F 2 "" H 13550 5500 50  0001 C CNN
